File: Hardware/MAIN_MODULE/MAIN_MODULE.brd (EAGLE design)
At the start: 100 x 80 mm, 14 parts

Commit message: Add files via upload
Parts:
- removed P_MM1, P_MM2, P_MM3, P_MM4: (no value), pinhead:2X10
- added <P_MM1, <P_MM4, P_MM2>, P_MM3>: (no value), pinhead:2X10
- moved P2 1.80 mm to (49.5, 40.6)
- moved P3 1.27 mm to (26.7, 63.5)
Connections:
- net FPGA_112: now also P_MM3>.3; no longer P_MM3.3
- net FPGA_113: now also P_MM3>.4; no longer P_MM3.4
- net FPGA_114: now also P_MM3>.5; no longer P_MM3.5
- net FPGA_115: now also P_MM3>.6; no longer P_MM3.6
- net FPGA_118: now also P_MM3>.7; no longer P_MM3.7
- net FPGA_119: now also P_MM3>.8; no longer P_MM3.8
- net FPGA_120: now also P_MM3>.9; no longer P_MM3.9
- net FPGA_121: now also P_MM3>.10; no longer P_MM3.10
- net FPGA_122: now also P_MM3>.11; no longer P_MM3.11
- net FPGA_125: now also P_MM3>.12; no longer P_MM3.12
- net FPGA_126: now also P_MM3>.13; no longer P_MM3.13
- net FPGA_129: now also P_MM3>.14; no longer P_MM3.14
- net FPGA_132: now also P_MM3>.15; no longer P_MM3.15
- net FPGA_133: now also P_MM3>.16; no longer P_MM3.16
- net FPGA_134: now also P_MM3>.17; no longer P_MM3.17
- net FPGA_135: now also P_MM3>.18; no longer P_MM3.18
- net FPGA_141: now also <P_MM4.3; no longer P_MM4.3
- net FPGA_142: now also <P_MM4.4; no longer P_MM4.4
- net FPGA_143: now also <P_MM4.5; no longer P_MM4.5
- net FPGA_18: now also <P_MM4.8; no longer P_MM4.8
- net FPGA_21: now also <P_MM4.10; no longer P_MM4.10
- net FPGA_22: now also <P_MM4.9; no longer P_MM4.9
- net FPGA_24: now also <P_MM4.12; no longer P_MM4.12
- net FPGA_25: now also <P_MM4.11; no longer P_MM4.11
- net FPGA_26: now also <P_MM4.14; no longer P_MM4.14
- net FPGA_27: now also <P_MM4.13; no longer P_MM4.13
- net FPGA_28: now also <P_MM4.16; no longer P_MM4.16
- net FPGA_30: now also <P_MM4.15; no longer P_MM4.15
- net FPGA_31: now also <P_MM4.18; no longer P_MM4.18
- net FPGA_32: now also <P_MM4.17; no longer P_MM4.17
- net FPGA_4: now also <P_MM4.6; no longer P_MM4.6
- net FPGA_40: now also <P_MM1.3; no longer P_MM1.3
- net FPGA_41: now also <P_MM1.4; no longer P_MM1.4
- net FPGA_42: now also <P_MM1.5; no longer P_MM1.5
- net FPGA_43: now also <P_MM1.6; no longer P_MM1.6
- net FPGA_44: now also <P_MM1.7; no longer P_MM1.7
- net FPGA_45: now also <P_MM1.8; no longer P_MM1.8
- net FPGA_47: now also <P_MM1.9; no longer P_MM1.9
- net FPGA_48: now also <P_MM1.10; no longer P_MM1.10
- net FPGA_51: now also <P_MM1.11; no longer P_MM1.11
- net FPGA_52: now also <P_MM1.12; no longer P_MM1.12
- net FPGA_53: now also <P_MM1.13; no longer P_MM1.13
- net FPGA_55: now also <P_MM1.14; no longer P_MM1.14
- net FPGA_57: now also <P_MM1.15; no longer P_MM1.15
- net FPGA_58: now also <P_MM1.16; no longer P_MM1.16
- net FPGA_59: now also <P_MM1.17; no longer P_MM1.17
- net FPGA_60: now also <P_MM1.18; no longer P_MM1.18
- net FPGA_73: now also P_MM2>.3; no longer P_MM2.3
- net FPGA_74: now also P_MM2>.4; no longer P_MM2.4
- net FPGA_75: now also P_MM2>.5; no longer P_MM2.5
- net FPGA_76: now also P_MM2>.6; no longer P_MM2.6
- net FPGA_79: now also P_MM2>.7; no longer P_MM2.7
- net FPGA_8: now also <P_MM4.7; no longer P_MM4.7
- net FPGA_80: now also P_MM2>.8; no longer P_MM2.8
- net FPGA_81: now also P_MM2>.9; no longer P_MM2.9
- net FPGA_86: now also P_MM2>.10; no longer P_MM2.10
- net FPGA_87: now also P_MM2>.11; no longer P_MM2.11
- net FPGA_88: now also P_MM2>.12; no longer P_MM2.12
- net FPGA_89: now also P_MM2>.13; no longer P_MM2.13
- net FPGA_90: now also P_MM2>.14; no longer P_MM2.14
- net FPGA_91: now also P_MM2>.15; no longer P_MM2.15
- net FPGA_92: now also P_MM2>.16; no longer P_MM2.16
- net FPGA_93: now also P_MM2>.17; no longer P_MM2.17
- net FPGA_94: now also P_MM2>.18; no longer P_MM2.18
- net FPGA_GND: now also <P_MM1.1, <P_MM1.20, <P_MM4.1, <P_MM4.20, P_MM2>.1, P_MM2>.20, P_MM3>.1, P_MM3>.20; no longer P_MM1.1, P_MM1.20, P_MM2.1, P_MM2.20, P_MM3.1, P_MM3.20, P_MM4.1, P_MM4.20
- net VIN: now also <P_MM1.19, <P_MM1.2, <P_MM4.19, <P_MM4.2, P_MM2>.19, P_MM2>.2, P_MM3>.19, P_MM3>.2; no longer P_MM1.19, P_MM1.2, P_MM2.19, P_MM2.2, P_MM3.19, P_MM3.2, P_MM4.19, P_MM4.2
Routing:
- net FPGA_GND: track 487.0 -> 404.1 mm, vias 4 -> 3
- net FPGA_135: track 86.8 -> 143.5 mm, vias 2 -> 5
- net FPGA_136: track 55.0 -> 99.7 mm, vias 3 -> 6
- net FPGA_129: track 108.1 -> 70.6 mm, vias 4 -> 2
- net FPGA_133: track 65.6 -> 100.5 mm, vias 4 -> 3
- net FPGA_26: track 56.0 -> 87.5 mm
- net FPGA_92: track 81.3 -> 109.8 mm
- net FPGA_103: track 56.6 -> 31.8 mm, vias 3 -> 2
- net VIN: track 347.2 -> 370.1 mm
- net FPGA_94: track 86.6 -> 109.4 mm, vias 1 -> 2
- net FPGA_48: track 18.2 -> 40.4 mm
- net FPGA_119: track 103.7 -> 84.2 mm
- net FPGA_120: track 71.3 -> 90.6 mm, vias 1 -> 2
- net FPGA_24: track 49.8 -> 67.1 mm, vias 6 -> 3
- net FPGA_28: track 81.0 -> 64.3 mm, vias 4 -> 2
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Other:
- outline, holes or cut-outs redrawn
- board text added: "D0"
- board text added: "D1"
- board text added: "FPGA"
- board text added: "MAIN MODULE v 1.1"
- board text added: "RXD"
- board text added: "TXD"
- board text removed: "MAIN MODULE v 1.0"
- board text removed: "RXD/D0"
- board text removed: "TXD/D1"

Commit message: Add files via upload
Parts:
- added JP2: (no value), pinhead:1X02
- moved <P_MM4 3.59 mm to (19.1, 73.7)
- moved <P_MM1 3.59 mm to (19.1, 6.35)
- moved P_MM3> 3.59 mm to (81.3, 73.7)
- moved P_MM2> 3.59 mm to (81.3, 6.35)
Connections:
- new net FPGA_144: P3.25
- net FPGA_112: now also P_MM2>.9
- net FPGA_40: now also P_MM2>.6
- net FPGA_73: now also P_MM2>.12
- net FPGA_76: no longer P_MM2>.6
- net FPGA_80: no longer P_MM2>.8
- net FPGA_81: no longer P_MM2>.9
- net FPGA_88: now also P_MM2>.8; no longer P_MM2>.12
- net FPGA_GND: now also JP2.2; no longer P3.25
- net VCC: now also JP2.1
Routing:
- net FPGA_112: track 62.8 -> 155.7 mm, vias 3 -> 1
- net FPGA_135: track 143.5 -> 61.1 mm, vias 5 -> 3
- net VIN: track 370.1 -> 288.9 mm, vias 3 -> 2
- net FPGA_40: track 15.0 -> 79.4 mm
- net FPGA_80: track 61.2 -> 0.00 mm, vias 1 -> 0
- net FPGA_81: track 56.9 -> 0.00 mm
- net FPGA_136: track 99.7 -> 54.0 mm, vias 6 -> 3
- net FPGA_76: track 45.3 -> 0.00 mm, vias 3 -> 0
- net FPGA_133: track 100.5 -> 57.9 mm, vias 3 -> 2
- net FPGA_92: track 109.8 -> 69.0 mm
- net FPGA_94: track 109.4 -> 71.6 mm, vias 2 -> 0
- net FPGA_125: track 59.8 -> 96.4 mm, vias 2 -> 3
- net FPGA_126: track 59.5 -> 94.2 mm, vias 1 -> 2
- net FPGA_69: track 88.3 -> 121.6 mm
- net FPGA_72: track 71.3 -> 100.5 mm, vias 4 -> 2
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Other:
- board text added: "MAIN MODULE v 1.2"
- board text removed: "MAIN MODULE v 1.1"

Commit message: Add files via upload
Parts:
- removed SA_A: (no value), pinhead:1X06
- removed SA_D1, SA_P: (no value), pinhead:1X08
- removed SA_D2: (no value), pinhead:1X10
- added JP3: (no value), pinhead:1X02
- added U$1, U$2, U$3, U$4: ST2378E_TSSOP, ST2378E:TSSOP20
- <P_MM1, <P_MM4, P_MM2>, P_MM3>: device pinhead:2X10 -> pinhead:2X05
- moved <P_MM4 1.80 mm to (17.8, 74.9), turned to 180 degrees
- moved P_MM3> 1.80 mm to (82.5, 74.9)
- moved <P_MM1 1.80 mm to (17.8, 5.08)
- moved P_MM2> 1.80 mm to (82.5, 5.08)
Connections:
- removed net AD0: SA_A.1
- removed net AD1: SA_A.2
- removed net AD2: SA_A.3
- removed net AD3: SA_A.4
- removed net AD4: SA_A.5, SA_D2.9
- removed net AD5: SA_A.6, SA_D2.10
- removed net AREF: SA_D2.8
- removed net NC: SA_P.1
- removed net RST: SA_P.3
- new net AR1_D0: <P_MM1.3, U$1.19
- new net AR1_D1: <P_MM1.4, U$1.3
- new net AR1_D12: <P_MM1.9, U$1.13
- new net AR1_D13: <P_MM1.10, U$1.P$9
- new net AR1_D2: <P_MM1.5, U$1.17
- new net AR1_D4: <P_MM1.6, U$1.5
- new net AR1_D7: <P_MM1.7, U$1.15
- new net AR1_D8: <P_MM1.8, U$1.7
- new net AR2_D0: P_MM2>.3, U$2.19
- new net AR2_D1: P_MM2>.4, U$2.3
- new net AR2_D12: P_MM2>.9, U$2.13
- new net AR2_D13: P_MM2>.10, U$2.P$9
- new net AR2_D2: P_MM2>.5, U$2.17
- new net AR2_D4: P_MM2>.6, U$2.5
- new net AR2_D7: P_MM2>.7, U$2.15
- new net AR2_D8: P_MM2>.8, U$2.7
- new net AR3_D0: P_MM3>.3, U$3.19
- new net AR3_D1: P_MM3>.4, U$3.3
- new net AR3_D12: P_MM3>.9, U$3.13
- new net AR3_D13: P_MM3>.10, U$3.P$9
- new net AR3_D2: P_MM3>.5, U$3.17
- new net AR3_D4: P_MM3>.6, U$3.5
- new net AR3_D7: P_MM3>.7, U$3.15
- new net AR3_D8: P_MM3>.8, U$3.7
- new net AR4_D0: <P_MM4.3, U$4.19
- new net AR4_D1: <P_MM4.4, U$4.3
- new net AR4_D12: <P_MM4.9, U$4.13
- new net AR4_D13: <P_MM4.10, U$4.P$9
- new net AR4_D2: <P_MM4.5, U$4.17
- new net AR4_D4: <P_MM4.6, U$4.5
- new net AR4_D7: <P_MM4.7, U$4.15
- new net AR4_D8: <P_MM4.8, U$4.7
- net FPGA_100: no longer SA_D2.4
- net FPGA_101: no longer SA_D2.5
- net FPGA_112: now also U$3.2; no longer P_MM2>.9, P_MM3>.3
- net FPGA_113: now also U$3.18; no longer P_MM3>.4
- net FPGA_114: now also U$3.4; no longer P_MM3>.5
- net FPGA_115: now also U$3.16; no longer P_MM3>.6
- net FPGA_118: now also U$3.6; no longer P_MM3>.7
- net FPGA_119: no longer P_MM3>.8
- net FPGA_120: now also U$3.8; no longer P_MM3>.9
- net FPGA_121: now also U$3.14; no longer P_MM3>.10
- net FPGA_122: no longer P_MM3>.11
- net FPGA_125: now also U$3.12; no longer P_MM3>.12
- net FPGA_126: now also U$3.11; no longer P_MM3>.13
- net FPGA_129: no longer P_MM3>.14
- net FPGA_132: no longer P_MM3>.15
- net FPGA_133: no longer P_MM3>.16
- net FPGA_134: no longer P_MM3>.17
- net FPGA_135: no longer P_MM3>.18
- net FPGA_136: no longer SA_D2.6
- net FPGA_141: now also U$4.2; no longer <P_MM4.3
- net FPGA_142: now also U$4.18; no longer <P_MM4.4
- net FPGA_143: now also U$4.4; no longer <P_MM4.5
- net FPGA_18: now also U$4.14; no longer <P_MM4.8
- net FPGA_21: now also U$4.12; no longer <P_MM4.10
- net FPGA_22: now also U$4.8; no longer <P_MM4.9
- net FPGA_24: no longer <P_MM4.12
- net FPGA_25: now also U$4.11; no longer <P_MM4.11
- net FPGA_26: no longer <P_MM4.14
- net FPGA_27: no longer <P_MM4.13
- net FPGA_28: no longer <P_MM4.16
- net FPGA_30: no longer <P_MM4.15
- net FPGA_31: no longer <P_MM4.18
- net FPGA_32: no longer <P_MM4.17
- net FPGA_4: now also U$4.16; no longer <P_MM4.6
- net FPGA_40: now also U$1.2; no longer <P_MM1.3, P_MM2>.6
- net FPGA_41: now also U$1.18; no longer <P_MM1.4
- net FPGA_42: now also U$1.4; no longer <P_MM1.5
- net FPGA_43: now also U$1.16; no longer <P_MM1.6
- net FPGA_44: now also U$1.6; no longer <P_MM1.7
- net FPGA_45: now also U$1.14; no longer <P_MM1.8
- net FPGA_47: now also U$1.8; no longer <P_MM1.9
- net FPGA_48: now also U$1.12; no longer <P_MM1.10
- net FPGA_51: now also U$1.11; no longer <P_MM1.11
- net FPGA_52: no longer <P_MM1.12
- net FPGA_53: no longer <P_MM1.13
- net FPGA_55: no longer <P_MM1.14
- net FPGA_57: no longer <P_MM1.15
- net FPGA_58: no longer <P_MM1.16
- net FPGA_59: no longer <P_MM1.17
- net FPGA_60: no longer <P_MM1.18
- net FPGA_63: no longer SA_D1.1
- net FPGA_64: no longer SA_D1.2
- net FPGA_65: no longer SA_D1.3
- net FPGA_67: no longer SA_D1.4
- net FPGA_69: no longer SA_D1.5
- net FPGA_70: no longer SA_D1.6
- net FPGA_71: no longer SA_D1.7
- net FPGA_72: no longer SA_D1.8
- net FPGA_73: now also U$2.2; no longer P_MM2>.12, P_MM2>.3
- net FPGA_74: now also U$2.18; no longer P_MM2>.4
- net FPGA_75: now also U$2.4; no longer P_MM2>.5
- net FPGA_79: now also U$2.6; no longer P_MM2>.7
- net FPGA_8: now also U$4.6; no longer <P_MM4.7
- net FPGA_86: now also U$2.14; no longer P_MM2>.10
- net FPGA_87: now also U$2.8; no longer P_MM2>.11
- net FPGA_88: now also U$2.12, U$2.16; no longer P_MM2>.8
- net FPGA_89: now also U$2.11; no longer P_MM2>.13
- net FPGA_90: no longer P_MM2>.14
- net FPGA_91: no longer P_MM2>.15
- net FPGA_92: no longer P_MM2>.16
- net FPGA_93: no longer P_MM2>.17
- net FPGA_94: no longer P_MM2>.18
- net FPGA_96: no longer SA_D2.1
- net FPGA_97: no longer SA_D2.2
- net FPGA_99: no longer SA_D2.3
- net FPGA_GND: now also JP3.2, U$1.P$10, U$2.P$10, U$3.P$10, U$4.P$10; no longer <P_MM1.20, <P_MM4.20, P_MM2>.20, P_MM3>.20, SA_D2.7, SA_P.6, SA_P.7
- net FPGA_VCC: now also U$1.1, U$2.1, U$3.1, U$4.1; no longer SA_P.4
- net VCC: now also JP3.1, U$1.20, U$2.20, U$3.20, U$4.20; no longer SA_P.2, SA_P.5
- net VIN: no longer <P_MM1.19, <P_MM4.19, P_MM2>.19, P_MM3>.19, SA_P.8
Routing:
- net VCC: track 25.8 -> 218.2 mm, vias 0 -> 3
- net FPGA_69: track 121.6 -> 0.00 mm, vias 2 -> 0
- net FPGA_112: track 155.7 -> 45.7 mm, vias 1 -> 3
- net FPGA_72: track 100.5 -> 0.00 mm, vias 2 -> 0
- net FPGA_63: track 99.9 -> 0.00 mm, vias 4 -> 0
- net FPGA_65: track 94.1 -> 0.00 mm, vias 3 -> 0
- net FPGA_67: track 90.2 -> 0.00 mm, vias 2 -> 0
- net FPGA_134: track 87.7 -> 0.00 mm, vias 3 -> 0
- net FPGA_70: track 87.5 -> 0.00 mm, vias 3 -> 0
- net FPGA_64: track 87.1 -> 0.00 mm, vias 1 -> 0
- net FPGA_VCC: track 146.0 -> 233.0 mm, vias 2 -> 3
- net FPGA_71: track 85.5 -> 0.00 mm, vias 4 -> 0
- net FPGA_91: track 80.4 -> 0.00 mm, vias 1 -> 0
- net FPGA_31: track 80.2 -> 0.00 mm, vias 3 -> 0
- net FPGA_122: track 78.4 -> 0.00 mm, vias 4 -> 0
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Other:
- board text added: "MAIN MODULE v 1.3"
- board text removed: "3V3"
- board text removed: "AD0"
- board text removed: "AD1"
- board text removed: "AD2"
- board text removed: "AD3"
- board text removed: "AD4"
- board text removed: "AD5"
- board text removed: "AREF"
- board text removed: "D0"
- board text removed: "D1"
- board text removed: "D10"
- board text removed: "D11"
- board text removed: "D12"
- board text removed: "D13"
- board text removed: "D2"
- board text removed: "D3"
- board text removed: "D4"
- board text removed: "D5"
- board text removed: "D6"
- board text removed: "D7"
- board text removed: "D8"
- board text removed: "D9"
- board text removed: "IOREF"
- board text removed: "MAIN MODULE v 1.2"
- board text removed: "P"
- board text removed: "R"
- board text removed: "RST"
- board text removed: "RXD"
- board text removed: "TXD"
