File: Hardware/MAIN_MODULE/MAIN_MODULE.sch (EAGLE design)
At the start: 14 parts

Commit message: Add files via upload
Parts:
- renumbered P_MM1 to <P_MM1, P_MM2 to P_MM2>, P_MM3 to P_MM3>, P_MM4 to <P_MM4

Commit message: Add files via upload
Parts:
- added JP2: (no value), pinhead:PINHD-1X2
Connections:
- new net FPGA_144: P3.25
- net FPGA_112: now also P_MM2>.9
- net FPGA_40: now also P_MM2>.6
- net FPGA_73: now also P_MM2>.12
- net FPGA_76: no longer P_MM2>.6
- net FPGA_80: no longer P_MM2>.8
- net FPGA_81: no longer P_MM2>.9
- net FPGA_88: now also P_MM2>.8; no longer P_MM2>.12
- net FPGA_GND: now also JP2.2; no longer P3.25
- net VCC: now also JP2.1

Commit message: Add files via upload
Parts:
- removed SA_A: (no value), pinhead:PINHD-1X6
- removed SA_D1, SA_P: (no value), pinhead:PINHD-1X8
- removed SA_D2: (no value), pinhead:PINHD-1X10
- added JP3: (no value), pinhead:PINHD-1X2
- added U$1, U$2, U$3, U$4: ST2378E_TSSOP, ST2378E:ST2378E_TSSOP
- <P_MM1, <P_MM4, P_MM2>, P_MM3>: device pinhead:PINHD-2X10 -> pinhead:PINHD-2X5
Connections:
- removed net AD0: SA_A.1
- removed net AD1: SA_A.2
- removed net AD2: SA_A.3
- removed net AD3: SA_A.4
- removed net AD4: SA_A.5, SA_D2.9
- removed net AD5: SA_A.6, SA_D2.10
- removed net AREF: SA_D2.8
- removed net NC: SA_P.1
- removed net RST: SA_P.3
- new net AR1_D0: <P_MM1.3, U$1.I/O_1_H
- new net AR1_D1: <P_MM1.4, U$1.I/O_2_H
- new net AR1_D12: <P_MM1.9, U$1.I/O_7_H
- new net AR1_D13: <P_MM1.10, U$1.I/O_8_H
- new net AR1_D2: <P_MM1.5, U$1.I/O_3_H
- new net AR1_D4: <P_MM1.6, U$1.I/O_4_H
- new net AR1_D7: <P_MM1.7, U$1.I/O_5_H
- new net AR1_D8: <P_MM1.8, U$1.I/O_6_H
- new net AR2_D0: P_MM2>.3, U$2.I/O_1_H
- new net AR2_D1: P_MM2>.4, U$2.I/O_2_H
- new net AR2_D12: P_MM2>.9, U$2.I/O_7_H
- new net AR2_D13: P_MM2>.10, U$2.I/O_8_H
- new net AR2_D2: P_MM2>.5, U$2.I/O_3_H
- new net AR2_D4: P_MM2>.6, U$2.I/O_4_H
- new net AR2_D7: P_MM2>.7, U$2.I/O_5_H
- new net AR2_D8: P_MM2>.8, U$2.I/O_6_H
- new net AR3_D0: P_MM3>.3, U$3.I/O_1_H
- new net AR3_D1: P_MM3>.4, U$3.I/O_2_H
- new net AR3_D12: P_MM3>.9, U$3.I/O_7_H
- new net AR3_D13: P_MM3>.10, U$3.I/O_8_H
- new net AR3_D2: P_MM3>.5, U$3.I/O_3_H
- new net AR3_D4: P_MM3>.6, U$3.I/O_4_H
- new net AR3_D7: P_MM3>.7, U$3.I/O_5_H
- new net AR3_D8: P_MM3>.8, U$3.I/O_6_H
- new net AR4_D0: <P_MM4.3, U$4.I/O_1_H
- new net AR4_D1: <P_MM4.4, U$4.I/O_2_H
- new net AR4_D12: <P_MM4.9, U$4.I/O_7_H
- new net AR4_D13: <P_MM4.10, U$4.I/O_8_H
- new net AR4_D2: <P_MM4.5, U$4.I/O_3_H
- new net AR4_D4: <P_MM4.6, U$4.I/O_4_H
- new net AR4_D7: <P_MM4.7, U$4.I/O_5_H
- new net AR4_D8: <P_MM4.8, U$4.I/O_6_H
- net FPGA_100: no longer SA_D2.4
- net FPGA_101: no longer SA_D2.5
- net FPGA_112: now also U$3.I/O_1_L; no longer P_MM2>.9, P_MM3>.3
- net FPGA_113: now also U$3.I/O_2_L; no longer P_MM3>.4
- net FPGA_114: now also U$3.I/O_3_L; no longer P_MM3>.5
- net FPGA_115: now also U$3.I/O_4_L; no longer P_MM3>.6
- net FPGA_118: now also U$3.I/O_5_L; no longer P_MM3>.7
- net FPGA_119: no longer P_MM3>.8
- net FPGA_120: now also U$3.I/O_7_L; no longer P_MM3>.9
- net FPGA_121: now also U$3.I/O_6_L; no longer P_MM3>.10
- net FPGA_122: no longer P_MM3>.11
- net FPGA_125: now also U$3.I/O_8_L; no longer P_MM3>.12
- net FPGA_126: now also U$3.OE; no longer P_MM3>.13
- net FPGA_129: no longer P_MM3>.14
- net FPGA_132: no longer P_MM3>.15
- net FPGA_133: no longer P_MM3>.16
- net FPGA_134: no longer P_MM3>.17
- net FPGA_135: no longer P_MM3>.18
- net FPGA_136: no longer SA_D2.6
- net FPGA_141: now also U$4.I/O_1_L; no longer <P_MM4.3
- net FPGA_142: now also U$4.I/O_2_L; no longer <P_MM4.4
- net FPGA_143: now also U$4.I/O_3_L; no longer <P_MM4.5
- net FPGA_18: now also U$4.I/O_6_L; no longer <P_MM4.8
- net FPGA_21: now also U$4.I/O_8_L; no longer <P_MM4.10
- net FPGA_22: now also U$4.I/O_7_L; no longer <P_MM4.9
- net FPGA_24: no longer <P_MM4.12
- net FPGA_25: now also U$4.OE; no longer <P_MM4.11
- net FPGA_26: no longer <P_MM4.14
- net FPGA_27: no longer <P_MM4.13
- net FPGA_28: no longer <P_MM4.16
- net FPGA_30: no longer <P_MM4.15
- net FPGA_31: no longer <P_MM4.18
- net FPGA_32: no longer <P_MM4.17
- net FPGA_4: now also U$4.I/O_4_L; no longer <P_MM4.6
- net FPGA_40: now also U$1.I/O_1_L; no longer <P_MM1.3, P_MM2>.6
- net FPGA_41: now also U$1.I/O_2_L; no longer <P_MM1.4
- net FPGA_42: now also U$1.I/O_3_L; no longer <P_MM1.5
- net FPGA_43: now also U$1.I/O_4_L; no longer <P_MM1.6
- net FPGA_44: now also U$1.I/O_5_L; no longer <P_MM1.7
- net FPGA_45: now also U$1.I/O_6_L; no longer <P_MM1.8
- net FPGA_47: now also U$1.I/O_7_L; no longer <P_MM1.9
- net FPGA_48: now also U$1.I/O_8_L; no longer <P_MM1.10
- net FPGA_51: now also U$1.OE; no longer <P_MM1.11
- net FPGA_52: no longer <P_MM1.12
- net FPGA_53: no longer <P_MM1.13
- net FPGA_55: no longer <P_MM1.14
- net FPGA_57: no longer <P_MM1.15
- net FPGA_58: no longer <P_MM1.16
- net FPGA_59: no longer <P_MM1.17
- net FPGA_60: no longer <P_MM1.18
- net FPGA_63: no longer SA_D1.1
- net FPGA_64: no longer SA_D1.2
- net FPGA_65: no longer SA_D1.3
- net FPGA_67: no longer SA_D1.4
- net FPGA_69: no longer SA_D1.5
- net FPGA_70: no longer SA_D1.6
- net FPGA_71: no longer SA_D1.7
- net FPGA_72: no longer SA_D1.8
- net FPGA_73: now also U$2.I/O_1_L; no longer P_MM2>.12, P_MM2>.3
- net FPGA_74: now also U$2.I/O_2_L; no longer P_MM2>.4
- net FPGA_75: now also U$2.I/O_3_L; no longer P_MM2>.5
- net FPGA_79: now also U$2.I/O_5_L; no longer P_MM2>.7
- net FPGA_8: now also U$4.I/O_5_L; no longer <P_MM4.7
- net FPGA_86: now also U$2.I/O_6_L; no longer P_MM2>.10
- net FPGA_87: now also U$2.I/O_7_L; no longer P_MM2>.11
- net FPGA_88: now also U$2.I/O_4_L, U$2.I/O_8_L; no longer P_MM2>.8
- net FPGA_89: now also U$2.OE; no longer P_MM2>.13
- net FPGA_90: no longer P_MM2>.14
- net FPGA_91: no longer P_MM2>.15
- net FPGA_92: no longer P_MM2>.16
- net FPGA_93: no longer P_MM2>.17
- net FPGA_94: no longer P_MM2>.18
- net FPGA_96: no longer SA_D2.1
- net FPGA_97: no longer SA_D2.2
- net FPGA_99: no longer SA_D2.3
- net FPGA_GND: now also JP3.2, U$1.GND, U$2.GND, U$3.GND, U$4.GND; no longer <P_MM1.20, <P_MM4.20, P_MM2>.20, P_MM3>.20, SA_D2.7, SA_P.6, SA_P.7
- net FPGA_VCC: now also U$1.VL, U$2.VL, U$3.VL, U$4.VL; no longer SA_P.4
- net VCC: now also JP3.1, U$1.VCC, U$2.VCC, U$3.VCC, U$4.VCC; no longer SA_P.2, SA_P.5
- net VIN: no longer <P_MM1.19, <P_MM4.19, P_MM2>.19, P_MM3>.19, SA_P.8
