File: Hardware/SECONDARY_MODULE/SECONDARY_MODULE.brd (EAGLE design)
At the start: 100 x 69.8 mm, 19 parts

Commit message: Add files via upload
Parts:
- moved D11 21.3 mm to (29.2, 5.08)
- moved AD5 17.7 mm to (78.7, 5.08)
- moved D10 17.7 mm to (25.4, 5.08)
- moved D9 14.2 mm to (21.6, 5.08)
- moved AD4 14.2 mm to (74.9, 5.08)
- moved SA_A 13.3 mm to (36.8, 17.8)
- moved SA_P 13.3 mm to (36.8, 38.1)
- moved NANO_D 12.5 mm to (25.4, 36.8)
- moved SA_D1 12.5 mm to (85.1, 20.3)
- moved SA_D2 12.5 mm to (85.1, 44.5)
- moved NANO_A 11.4 mm to (10.2, 36.8)
- moved AD3 10.9 mm to (71.1, 5.08)
- moved D6 10.9 mm to (17.8, 5.08)
- moved D5 8.13 mm to (14.0, 5.08)
- moved AD2 8.13 mm to (67.3, 5.08)
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Routing:
- net D10: track 214.5 -> 149.2 mm, vias 1 -> 2
- net D6: track 202.7 -> 141.2 mm, vias 1 -> 5
- net VCC: track 173.6 -> 131.1 mm, vias 2 -> 0
- net AD5: track 166.9 -> 198.1 mm
- net D8: track 130.3 -> 103.4 mm, vias 2 -> 1
- net AD4: track 207.4 -> 183.4 mm
- net D11: track 212.6 -> 188.9 mm, vias 1 -> 0
- net D3: track 146.5 -> 122.9 mm, vias 1 -> 3
- net GND: track 222.3 -> 201.8 mm, vias 1 -> 0
- net RST: track 84.0 -> 69.2 mm, vias 2 -> 0
- net D4: track 121.1 -> 108.0 mm, vias 1 -> 5
- net D12: track 114.8 -> 102.4 mm
- net D7: track 107.5 -> 95.8 mm, vias 1 -> 3
- net AD3: track 111.9 -> 100.6 mm
- net D13: track 118.0 -> 108.7 mm
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Other:
- board size 100 x 69.8 mm -> 93.7 x 58.4 mm
- board text added: "RX"
- board text added: "SECONDARY MODULE v1.1"
- board text added: "SIG"
- board text added: "TX"
- board text added: "VCC"
- board text removed: "D0/RX"
- board text removed: "D1/TX"
- board text removed: "SECONDARY MODULE v1.0"

Commit message: Add files via upload
Parts:
- added JP1: JP1, pinhead:1X04
- moved D11 5.08 mm to (24.1, 5.08)
- moved AD5 5.08 mm to (73.7, 5.08)
- moved AD4 3.81 mm to (71.1, 5.08)
- moved D10 3.81 mm to (21.6, 5.08)
- moved AD3 2.54 mm to (68.6, 5.08)
- moved D9 2.54 mm to (19.1, 5.08)
- moved AD0 1.27 mm to (61.0, 5.08)
- moved D3 1.27 mm to (11.4, 5.08)
- moved D6 1.27 mm to (16.5, 5.08)
- moved AD2 1.27 mm to (66.0, 5.08)
Connections:
- new net VCC_ENA: JP1.4
- new net VCC_SERVO: D10.2, D11.2, D3.2, D5.2, D6.2, D9.2, JP1.1
- net GND: now also JP1.2
- net VCC: no longer D10.2, D11.2, D3.2, D5.2, D6.2, D9.2
- net VIN: now also JP1.3
Routing:
- net D4: track 108.0 -> 218.1 mm, vias 5 -> 1
- net D11: track 188.9 -> 150.0 mm, vias 0 -> 1
- net AD5: track 198.1 -> 162.3 mm, vias 2 -> 3
- net VIN: track 70.2 -> 103.4 mm, vias 1 -> 2
- net VCC: track 131.1 -> 102.1 mm, vias 0 -> 1
- net VCC_SERVO: track 0.00 -> 26.7 mm
- net AD3: track 100.6 -> 126.2 mm, vias 2 -> 3
- net D3: track 122.9 -> 145.3 mm, vias 3 -> 5
- net AD1: track 91.3 -> 111.9 mm, vias 2 -> 1
- net D0: track 106.9 -> 92.1 mm, vias 1 -> 3
- net RST: track 69.2 -> 83.7 mm, vias 0 -> 2
- net D6: track 141.2 -> 152.5 mm, vias 5 -> 4
- net D13: track 108.7 -> 99.3 mm, vias 0 -> 1
- net D8: track 103.4 -> 94.7 mm
- net D2: track 99.8 -> 107.9 mm, vias 2 -> 3
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Other:
- board text added: "ENA"
- board text added: "SECONDARY MODULE v1.2"
- board text added: "VCC_SERVO"
- board text removed: "SECONDARY MODULE v1.1"

Commit message: Add files via upload
Parts:
- removed P_MM: P_MM, pinhead:2X10
- added JP2: (no value), pinhead:2X05
Connections:
- net D0: now also JP2.3; no longer P_MM.4
- net D1: now also JP2.4; no longer P_MM.5
- net D10: no longer P_MM.14
- net D11: no longer P_MM.15
- net D12: now also JP2.9; no longer P_MM.16
- net D13: now also JP2.10; no longer P_MM.17
- net D2: now also JP2.5; no longer P_MM.6
- net D3: no longer P_MM.7
- net D4: now also JP2.6; no longer P_MM.8
- net D5: no longer P_MM.9
- net D6: no longer P_MM.10
- net D7: now also JP2.7; no longer P_MM.11
- net D8: now also JP2.8; no longer P_MM.12
- net D9: no longer P_MM.13
- net GND: now also JP2.1; no longer P_MM.1, P_MM.20
- net RST: no longer P_MM.18, P_MM.3
- net VIN: now also JP2.2; no longer P_MM.19, P_MM.2
Routing:
- net D4: track 218.1 -> 145.9 mm, vias 1 -> 5
- net D7: track 101.9 -> 169.5 mm, vias 3 -> 6
- net D5: track 128.1 -> 185.4 mm, vias 4 -> 2
- net RST: track 83.7 -> 38.2 mm, vias 2 -> 0
- net AD4: track 184.2 -> 139.2 mm, vias 3 -> 7
- net AD1: track 111.9 -> 145.9 mm, vias 1 -> 5
- net D3: track 145.3 -> 115.9 mm, vias 5 -> 4
- net D9: track 140.8 -> 169.2 mm, vias 2 -> 0
- net D11: track 150.0 -> 175.5 mm, vias 1 -> 0
- net AD3: track 126.2 -> 102.1 mm, vias 3 -> 7
- net D10: track 154.7 -> 131.0 mm, vias 6 -> 2
- net D6: track 152.5 -> 173.9 mm, vias 4 -> 2
- net D2: track 107.9 -> 86.9 mm, vias 3 -> 0
- net GND: track 205.6 -> 184.7 mm, vias 0 -> 3
- net AD5: track 162.3 -> 181.1 mm, vias 3 -> 1
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Other:
- board text added: "SECONDARY MODULE v1.3"
- board text removed: "P"
- board text removed: "R"
- board text removed: "SECONDARY MODULE v1.2"
