File: Hardware/SECONDARY_MODULE/SECONDARY_MODULE.sch (EAGLE design)
At the start: 19 parts

Commit message: Add files via upload
Parts:
- added JP1: JP1, pinhead:PINHD-1X4
Connections:
- new net VCC_ENA: JP1.4
- new net VCC_SERVO: D10.2, D11.2, D3.2, D5.2, D6.2, D9.2, JP1.1
- net GND: now also JP1.2
- net VCC: no longer D10.2, D11.2, D3.2, D5.2, D6.2, D9.2
- net VIN: now also JP1.3
Changed lines of the file:
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@@
 <?xml version="1.0" encoding="utf-8"?>
 <!DOCTYPE eagle SYSTEM "eagle.dtd">
-<eagle version="7.5.0">
+<eagle version="8.0.0">
 <drawing>
 <settings>
@@
 <part name="NANO_D" library="pinhead" deviceset="PINHD-1X15" device="" value="NANO_D"/>
 <part name="NANO_A" library="pinhead" deviceset="PINHD-1X15" device="" value="NANO_A"/>
+<part name="JP1" library="pinhead" deviceset="PINHD-1X4" device="" value="JP1"/>
 </parts>
 <sheets>
@@
 <instance part="NANO_D" gate="A" x="43.18" y="99.06"/>
 <instance part="NANO_A" gate="A" x="50.8" y="99.06" rot="MR0"/>
+<instance part="JP1" gate="A" x="63.5" y="142.24"/>
 </instances>
 <busses>
@@
 </segment>
 <segment>
-<wire x1="134.62" y1="119.38" x2="121.92" y2="119.38" width="0.1524" layer="91"/>
-<label x="124.46" y="119.38" size="1.778" layer="95"/>
+<wire x1="134.62" y1="119.38" x2="116.84" y2="119.38" width="0.1524" layer="91"/>
+<label x="116.84" y="119.38" size="1.778" layer="95"/>
 <pinref part="D6" gate="A" pin="3"/>
 </segment>
@@
 </segment>
 <segment>
-<wire x1="134.62" y1="149.86" x2="121.92" y2="149.86" width="0.1524" layer="91"/>
-<label x="124.46" y="149.86" size="1.778" layer="95"/>
+<wire x1="134.62" y1="149.86" x2="116.84" y2="149.86" width="0.1524" layer="91"/>
+<label x="116.84" y="149.86" size="1.778" layer="95"/>
 <pinref part="D3" gate="A" pin="3"/>
 </segment>
@@
 </segment>
 <segment>
-<wire x1="134.62" y1="134.62" x2="121.92" y2="134.62" width="0.1524" layer="91"/>
-<label x="124.46" y="134.62" size="1.778" layer="95"/>
+<wire x1="134.62" y1="134.62" x2="116.84" y2="134.62" width="0.1524" layer="91"/>
+<label x="116.84" y="134.62" size="1.778" layer="95"/>
 <pinref part="D5" gate="A" pin="3"/>
 </segment>
@@
 </segment>
 <segment>
-<wire x1="134.62" y1="88.9" x2="121.92" y2="88.9" width="0.1524" layer="91"/>
-<label x="124.46" y="88.9" size="1.778" layer="95"/>
+<wire x1="134.62" y1="88.9" x2="116.84" y2="88.9" width="0.1524" layer="91"/>
+<label x="116.84" y="88.9" size="1.778" layer="95"/>
 <pinref part="D10" gate="A" pin="3"/>
 </segment>
@@
 </segment>
 <segment>
-<wire x1="134.62" y1="104.14" x2="121.92" y2="104.14" width="0.1524" layer="91"/>
-<label x="124.46" y="104.14" size="1.778" layer="95"/>
+<wire x1="134.62" y1="104.14" x2="116.84" y2="104.14" width="0.1524" layer="91"/>
+<label x="116.84" y="104.14" size="1.778" layer="95"/>
 <pinref part="D9" gate="A" pin="3"/>
 </segment>
@@
 </segment>
 <segment>
-<wire x1="134.62" y1="73.66" x2="121.92" y2="73.66" width="0.1524" layer="91"/>
-<label x="124.46" y="73.66" size="1.778" layer="95"/>
+<wire x1="134.62" y1="73.66" x2="116.84" y2="73.66" width="0.1524" layer="91"/>
+<label x="116.84" y="73.66" size="1.778" layer="95"/>
 <pinref part="D11" gate="A" pin="3"/>
 </segment>
@@
 <pinref part="NANO_A" gate="A" pin="1"/>
 </segment>
+<segment>
+<pinref part="JP1" gate="A" pin="3"/>
+<wire x1="60.96" y1="142.24" x2="40.64" y2="142.24" width="0.1524" layer="91"/>
+<label x="43.18" y="142.24" size="1.778" layer="95"/>
+</segment>
 </net>
 <net name="NC" class="0">
@@
 </segment>
 <segment>
-<wire x1="134.62" y1="152.4" x2="121.92" y2="152.4" width="0.1524" layer="91"/>
-<label x="124.46" y="152.4" size="1.778" layer="95"/>
-<pinref part="D3" gate="A" pin="2"/>
-</segment>
-<segment>
-<wire x1="134.62" y1="137.16" x2="121.92" y2="137.16" width="0.1524" layer="91"/>
-<label x="124.46" y="137.16" size="1.778" layer="95"/>
-<pinref part="D5" gate="A" pin="2"/>
-</segment>
-<segment>
-<wire x1="134.62" y1="121.92" x2="121.92" y2="121.92" width="0.1524" layer="91"/>
-<label x="124.46" y="121.92" size="1.778" layer="95"/>
-<pinref part="D6" gate="A" pin="2"/>
-</segment>
-<segment>
-<wire x1="134.62" y1="106.68" x2="121.92" y2="106.68" width="0.1524" layer="91"/>
-<label x="124.46" y="106.68" size="1.778" layer="95"/>
-<pinref part="D9" gate="A" pin="2"/>
-</segment>
-<segment>
-<wire x1="134.62" y1="91.44" x2="121.92" y2="91.44" width="0.1524" layer="91"/>
-<label x="124.46" y="91.44" size="1.778" layer="95"/>
-<pinref part="D10" gate="A" pin="2"/>
-</segment>
-<segment>
-<wire x1="134.62" y1="76.2" x2="121.92" y2="76.2" width="0.1524" layer="91"/>
-<label x="124.46" y="76.2" size="1.778" layer="95"/>
-<pinref part="D11" gate="A" pin="2"/>
-</segment>
-<segment>
 <wire x1="83.82" y1="152.4" x2="96.52" y2="152.4" width="0.1524" layer="91"/>
 <label x="91.44" y="152.4" size="1.778" layer="95"/>
@@
 </segment>
 <segment>
-<wire x1="134.62" y1="154.94" x2="121.92" y2="154.94" width="0.1524" layer="91"/>
-<label x="124.46" y="154.94" size="1.778" layer="95"/>
+<wire x1="134.62" y1="154.94" x2="116.84" y2="154.94" width="0.1524" layer="91"/>
+<label x="116.84" y="154.94" size="1.778" layer="95"/>
 <pinref part="D3" gate="A" pin="1"/>
 </segment>
 <segment>
-<wire x1="134.62" y1="139.7" x2="121.92" y2="139.7" width="0.1524" layer="91"/>
-<label x="124.46" y="139.7" size="1.778" layer="95"/>
+<wire x1="134.62" y1="139.7" x2="116.84" y2="139.7" width="0.1524" layer="91"/>
+<label x="116.84" y="139.7" size="1.778" layer="95"/>
 <pinref part="D5" gate="A" pin="1"/>
 </segment>
 <segment>
-<wire x1="134.62" y1="124.46" x2="121.92" y2="124.46" width="0.1524" layer="91"/>
-<label x="124.46" y="124.46" size="1.778" layer="95"/>
+<wire x1="134.62" y1="124.46" x2="116.84" y2="124.46" width="0.1524" layer="91"/>
+<label x="116.84" y="124.46" size="1.778" layer="95"/>
 <pinref part="D6" gate="A" pin="1"/>
 </segment>
 <segment>
-<wire x1="134.62" y1="109.22" x2="121.92" y2="109.22" width="0.1524" layer="91"/>
-<label x="124.46" y="109.22" size="1.778" layer="95"/>
+<wire x1="134.62" y1="109.22" x2="116.84" y2="109.22" width="0.1524" layer="91"/>
+<label x="116.84" y="109.22" size="1.778" layer="95"/>
 <pinref part="D9" gate="A" pin="1"/>
 </segment>
 <segment>
-<wire x1="134.62" y1="93.98" x2="121.92" y2="93.98" width="0.1524" layer="91"/>
-<label x="124.46" y="93.98" size="1.778" layer="95"/>
+<wire x1="134.62" y1="93.98" x2="116.84" y2="93.98" width="0.1524" layer="91"/>
+<label x="116.84" y="93.98" size="1.778" layer="95"/>
 <pinref part="D10" gate="A" pin="1"/>
 </segment>
 <segment>
-<wire x1="134.62" y1="78.74" x2="121.92" y2="78.74" width="0.1524" layer="91"/>
-<label x="124.46" y="78.74" size="1.778" layer="95"/>
+<wire x1="134.62" y1="78.74" x2="116.84" y2="78.74" width="0.1524" layer="91"/>
+<label x="116.84" y="78.74" size="1.778" layer="95"/>
 <pinref part="D11" gate="A" pin="1"/>
 </segment>
@@
 <pinref part="NANO_A" gate="A" pin="2"/>
 </segment>
+<segment>
+<pinref part="JP1" gate="A" pin="2"/>
+<wire x1="60.96" y1="144.78" x2="40.64" y2="144.78" width="0.1524" layer="91"/>
+<label x="43.18" y="144.78" size="1.778" layer="95"/>
+</segment>
 </net>
 <net name="AD7" class="0">
@@
 </segment>
 </net>
+<net name="VCC_SERVO" class="0">
+<segment>
+<pinref part="D3" gate="A" pin="2"/>
+<wire x1="134.62" y1="152.4" x2="116.84" y2="152.4" width="0.1524" layer="91"/>
+<label x="116.84" y="152.4" size="1.778" layer="95"/>
+</segment>
+<segment>
+<wire x1="134.62" y1="137.16" x2="116.84" y2="137.16" width="0.1524" layer="91"/>
+<label x="116.84" y="137.16" size="1.778" layer="95"/>
+<pinref part="D5" gate="A" pin="2"/>
+</segment>
+<segment>
+<wire x1="134.62" y1="121.92" x2="116.84" y2="121.92" width="0.1524" layer="91"/>
+<label x="116.84" y="121.92" size="1.778" layer="95"/>
+<pinref part="D6" gate="A" pin="2"/>
+</segment>
+<segment>
+<wire x1="134.62" y1="106.68" x2="116.84" y2="106.68" width="0.1524" layer="91"/>
+<label x="116.84" y="106.68" size="1.778" layer="95"/>
+<pinref part="D9" gate="A" pin="2"/>
+</segment>
+<segment>
+<wire x1="134.62" y1="91.44" x2="116.84" y2="91.44" width="0.1524" layer="91"/>
+<label x="116.84" y="91.44" size="1.778" layer="95"/>
+<pinref part="D10" gate="A" pin="2"/>
+</segment>
+<segment>
+<wire x1="134.62" y1="76.2" x2="116.84" y2="76.2" width="0.1524" layer="91"/>
+<label x="116.84" y="76.2" size="1.778" layer="95"/>
+<pinref part="D11" gate="A" pin="2"/>
+</segment>
+<segment>
+<pinref part="JP1" gate="A" pin="1"/>
+<wire x1="60.96" y1="147.32" x2="40.64" y2="147.32" width="0.1524" layer="91"/>
+<label x="43.18" y="147.32" size="1.778" layer="95"/>
+</segment>
+</net>
+<net name="VCC_ENA" class="0">
+<segment>
+<pinref part="JP1" gate="A" pin="4"/>
+<wire x1="60.96" y1="139.7" x2="40.64" y2="139.7" width="0.1524" layer="91"/>
+<label x="43.18" y="139.7" size="1.778" layer="95"/>
+</segment>
+</net>

Commit message: Add files via upload
Parts:
- removed P_MM: P_MM, pinhead:PINHD-2X10
- added JP2: (no value), pinhead:PINHD-2X5
Connections:
- net D0: now also JP2.3; no longer P_MM.4
- net D1: now also JP2.4; no longer P_MM.5
- net D10: no longer P_MM.14
- net D11: no longer P_MM.15
- net D12: now also JP2.9; no longer P_MM.16
- net D13: now also JP2.10; no longer P_MM.17
- net D2: now also JP2.5; no longer P_MM.6
- net D3: no longer P_MM.7
- net D4: now also JP2.6; no longer P_MM.8
- net D5: no longer P_MM.9
- net D6: no longer P_MM.10
- net D7: now also JP2.7; no longer P_MM.11
- net D8: now also JP2.8; no longer P_MM.12
- net D9: no longer P_MM.13
- net GND: now also JP2.1; no longer P_MM.1, P_MM.20
- net RST: no longer P_MM.18, P_MM.3
- net VIN: now also JP2.2; no longer P_MM.19, P_MM.2
